Commit message: Update thruster_ccw.xacro

File: nemo_description/urdf/thruster_ccw.xacro (robot description, xacro)
@@ -13,4 +13,10 @@
                          iyy="4.709701538508585e-06" iyz="0.0" izz="3.424149260721648e-06"/>
             </inertial>
+            <collision>
+                <origin xyz="0 0 0" rpy="0 0 0"/>
+                <geometry>
+                    <cylinder radius="0.09" length="0.05"/>
+                </geometry>
+            </collision>
         </link>
         <joint name="thruster${thruster_id}" type="continuous">
