Commit message: Update thruster_cw.xacro
Added Collision tags to fix the NaN error in Dart simulations

File: nemo_description/urdf/thruster_cw.xacro (robot description, xacro)
@@ -12,4 +12,10 @@
                 <inertia ixx="4.709701538510022e-06" ixy="0.0" ixz="0.0" iyy="4.709701538508585e-06" iyz="0.0" izz="3.424149260721648e-06"/>
             </inertial>
+            <collision>
+                <origin xyz="0 0 0" rpy="0 0 0"/>
+                <geometry>
+                    <cylinder radius="0.02" length="0.05"/>
+                </geometry>
+            </collision>
         </link>
         <joint name="thruster${thruster_id}" type="continuous">
@@ -18,5 +24,5 @@
             <parent link="base_link" />
             <child link="${ns}/thruster${thruster_id}" />
-            <limits effort="-1" velocity="-1"/>
+            <limits effort="0.5" velocity="5.0"/>
         </joint>
         <gazebo>
